File: vco_as3340_v1/vco_as3340_v1.kicad_pcb (KiCad board)
At the start: 2 copper layers, 49 x 100 mm, 88 parts, among them J100 FREQ_CV, J101 SYNC, J102 SAWTOOTH, J103 TRIANGLE, J104 PULSE, J2 Conn_02x05_Odd_Even, U1 LM7805_TO220, U2 L7905, U3 AS3340, U4 TL072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

Commit message: v2 re-layout pcb
Parts:
- removed C13, C17: 10nF, Capacitor_SMD:C_1206_3216Metric_Pad1.33x1.80mm_HandSolder
- removed FB1, FB2: FerriteBead, Inductor_THT:L_Axial_L6.6mm_D2.7mm_P2.54mm_Vertical_Vishay_IM-2
- removed JP1, JP2, JP3: Jumper_2_Open, Connector_PinHeader_2.54mm:PinHeader_1x02_P2.54mm_Vertical
- removed R5: 575, Resistor_SMD:R_1206_3216Metric_Pad1.30x1.75mm_HandSolder
- removed U5: TL072, Package_DIP:DIP-8_W7.62mm_Socket_LongPads
- added C1: 100pF, Capacitor_SMD:C_1206_3216Metric_Pad1.33x1.80mm_HandSolder, B.Cu at (173.9, 105.0)
- added C15: 10uF, Capacitor_THT:CP_Radial_D5.0mm_P2.50mm, B.Cu at (186.6, 106.9)
- added C19: 10nF, Capacitor_SMD:C_1206_3216Metric_Pad1.33x1.80mm_HandSolder, B.Cu at (151.0, 129.2)
- added C20: 10nF, Capacitor_SMD:C_1206_3216Metric_Pad1.33x1.80mm_HandSolder, B.Cu at (159.0, 75.5)
- added C21: 10nF, Capacitor_SMD:C_1206_3216Metric_Pad1.33x1.80mm_HandSolder, B.Cu at (165.0, 88.9)
- added JP5: Jumper_2_Bridged, Jumper:SolderJumper-2_P1.3mm_Bridged_Pad1.0x1.5mm, B.Cu at (157.5, 103.1)
- added JP6: Jumper_3_Bridged12, Jumper:SolderJumper-3_P1.3mm_Bridged12_Pad1.0x1.5mm, B.Cu at (166.5, 75.1)
- added R31: 100k, Resistor_SMD:R_1206_3216Metric_Pad1.30x1.75mm_HandSolder, B.Cu at (183.4, 116.9)
- added R32: 2M, Resistor_SMD:R_1206_3216Metric_Pad1.30x1.75mm_HandSolder, B.Cu at (171.3, 101.2)
- added R33: DNU, Resistor_SMD:R_1206_3216Metric_Pad1.30x1.75mm_HandSolder, B.Cu at (157.8, 85.1)
- added R34: 0, Resistor_SMD:R_1206_3216Metric_Pad1.30x1.75mm_HandSolder, B.Cu at (157.8, 80.0)
- added R35: 100k, Resistor_SMD:R_1206_3216Metric_Pad1.30x1.75mm_HandSolder, B.Cu at (171.3, 84.6)
- added R36: 100k, Resistor_SMD:R_1206_3216Metric_Pad1.30x1.75mm_HandSolder, B.Cu at (171.3, 79.4)
- added R37: 51k, Resistor_SMD:R_1206_3216Metric_Pad1.30x1.75mm_HandSolder, B.Cu at (143.3, 107.8)
- added R38: 100k, Resistor_SMD:R_1206_3216Metric_Pad1.30x1.75mm_HandSolder, B.Cu at (144.7, 68.9)
- added R39: 100k, Resistor_SMD:R_1206_3216Metric_Pad1.30x1.75mm_HandSolder, B.Cu at (149.9, 68.9)
- added REF_PITCH2: 100k, Potentiometer_THT:Potentiometer_Bourns_3296W_Vertical, F.Cu at (148.2, 65.9)
- added REF_VOLT_1: 100k, Potentiometer_THT:Potentiometer_Bourns_3296W_Vertical, F.Cu at (148.3, 111.4)
- added TP3: REF_VOLT_1, Connector_PinHeader_2.54mm:PinHeader_1x01_P2.54mm_Vertical, B.Cu at (169.5, 89.8)
- added TP4: REF_VOLT_2, Connector_PinHeader_2.54mm:PinHeader_1x01_P2.54mm_Vertical, B.Cu at (171.0, 75.1)
- added U6: TL072, Package_DIP:DIP-8_W7.62mm_Socket_LongPads, B.Cu at (168.3, 78.4)
- C10, C11, C12, C16, C18, C3, C6, C7, C8, C9: moved to B.Cu
- HF_TRACK1, REFIND_C6, REF_PITCH1, RZ_TEMP1, SCALE_ADJ1: moved to F.Cu
- R10: value 50k -> 47k
- R21, R23: value 5k -> 5.1k
- R26: value 200k -> 100k
- R6: value 100k -> DNU
- R9: value 1k -> 0
- RZ1: value 13k -> 18k
- U4: value TL072 -> TL074; footprint Package_DIP:DIP-8_W7.62mm_Socket_LongPads -> Package_DIP:DIP-14_W7.62mm_Socket_LongPads
- moved LOGO1 96.8 mm to (88.7, 141.8)
- moved LOGO2 87.7 mm to (101.3, 130.8)
- moved LOGO101 61.5 mm to (89.8, 123.8)
- moved Rs2 52.5 mm to (153.8, 53.0)
- moved Rs1 50.6 mm to (157.8, 54.6), turned to 90 degrees
- moved C5 43.0 mm to (153.8, 56.3), turned to 0 degrees
- moved C14 38.2 mm to (175.1, 85.9)
- moved R12 35.5 mm to (175.1, 83.4), turned to 180 degrees
- moved Rr2 31.1 mm to (175.2, 78.5)
- moved R6 29.6 mm to (183.3, 126.9)
- moved R13 27.2 mm to (167.1, 132.1)
- moved R20 25.2 mm to (161.7, 114.4), turned to 0 degrees
- moved Rr1 25.0 mm to (175.2, 80.9), turned to 0 degrees
- moved R15 23.3 mm to (166.7, 137.5), turned to 0 degrees
- moved SCALE_ADJ1 22.2 mm to (148.2, 53.3), turned to 0 degrees
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Connections:
- net /Outputs/Pulse Output renamed /Inputs/To Pulse
- C10 pad 1: -12V -> -5V
- D1 pad 2: Net-(D1-Pad2) -> -12V
- D2 pad 1: Net-(D2-Pad1) -> +12V
- R14 pad 2: Net-(R15-Pad1) -> Net-(R14-Pad2)
- R15 pad 1: Net-(R15-Pad1) -> Net-(R14-Pad2)
- R16 pad 1: Net-(R17-Pad2) -> Net-(R16-Pad1)
- R17 pad 2: Net-(R17-Pad2) -> Net-(R16-Pad1)
- R2 pad 1: Net-(JP1-Pad1) -> /Inputs/Frequency Control
- R24 pad 2: Net-(R26-Pad1) -> Net-(R24-Pad2)
- R26 pad 1: Net-(R26-Pad1) -> Net-(R24-Pad2)
- R27 pad 1: Net-(R29-Pad1) -> Net-(R27-Pad1)
- R28 pad 1: Net-(R26-Pad2) -> Net-(R28-Pad1)
- R29 pad 1: Net-(R29-Pad1) -> Net-(R27-Pad1)
- R3 pad 1: Net-(JP1-Pad1) -> /Inputs/Frequency Control
- R6 pad 2: Net-(R8-Pad1) -> Net-(R6-Pad2)
- R7 pad 2: Net-(R8-Pad1) -> Net-(R6-Pad2)
- R8 pad 1: Net-(R8-Pad1) -> Net-(R6-Pad2)
- REF_PITCH1 pad 1: Net-(R4-Pad1) -> +12V
- REF_PITCH1 pad 2: Net-(REF_PITCH1-Pad2) -> Net-(JP6-Pad3)
- REF_PITCH1 pad 3: +12V -> Net-(R4-Pad1)
- Rr2 pad 2: Net-(REF_PITCH1-Pad2) -> Net-(JP6-Pad2)
- U3 pad 3: VEE -> -5V
- U4 pad 1: Net-(R11-Pad1) -> Net-(R28-Pad1)
- U4 pad 2: Net-(R17-Pad2) -> Net-(R24-Pad2)
- U4 pad 3: GND -> /Outputs/Triangle Output
- U4 pad 4: -12V -> +12V
- U4 pad 5: GND -> Net-(R6-Pad2)
- U4 pad 6: Net-(R11-Pad2) -> Net-(R25-Pad1)
- U4 pad 7: Net-(R15-Pad1) -> Net-(R27-Pad1)
- U4 pad 8: +12V -> Net-(R11-Pad1)
Routing:
- net +12V: track 175.1 -> 0.00 mm, vias 2 -> 0
- net -12V: track 111.7 -> 0.00 mm, vias 2 -> 0
- net /Inputs/Frequency Control: track 100.5 -> 0.00 mm, vias 2 -> 0
- net +5V: track 70.1 -> 0.00 mm
- net Net-(JP1-Pad1): track 49.3 -> 0.00 mm
- net Net-(R8-Pad1): track 41.7 -> 0.00 mm, vias 2 -> 0
- net /Inputs/Hard Sync: track 39.1 -> 0.00 mm, vias 1 -> 0
- net /Outputs/Triangle Output: track 37.2 -> 0.00 mm
- net VEE: track 34.9 -> 0.00 mm
- net /Inputs/PWM Control: track 33.5 -> 0.00 mm, vias 1 -> 0
- net Net-(R11-Pad2): track 32.7 -> 0.00 mm
- net Net-(Rs2-Pad2): track 32.1 -> 0.00 mm
- net /Outputs/Sawtooth Output: track 30.2 -> 0.00 mm
- net Net-(J102-PadT): track 28.1 -> 0.00 mm, vias 1 -> 0
- net /Inputs/Scale Adjust 2: track 26.7 -> 0.00 mm
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Other:
- board text added: "move pots to front"
- board text added: "v2.0 Nov 2022"
- board text removed: "v1.0 July 2022"

Commit message: Routing done
Parts:
- removed JP6: Jumper_3_Bridged12, Jumper:SolderJumper-3_P1.3mm_Bridged12_Pad1.0x1.5mm
- removed the REF_PITCH1 at (148.2, 72.2)
- added J1: FREQ_CV2, My Stuff:Jack_3.5mm_MJ-355W_Vertical, F.Cu at (145.4, 131.0)
- added R5: 100k,0.05%, Resistor_SMD:R_1206_3216Metric_Pad1.30x1.75mm_HandSolder, B.Cu at (147.0, 130.5)
- R4: value 22k -> 0
- REF_PITCH1: renamed from REF_PITCH2; moved to B.Cu
- REF_VOLT_1, RZ_TEMP1: moved to B.Cu
- TP4: value REF_VOLT_2 -> REF_PITCH_1
- moved LOGO101 96.1 mm to (164.5, 63.3), turned to 0 degrees
- moved LOGO1 85.3 mm to (164.5, 102.6)
- moved LOGO2 80.2 mm to (145.9, 64.1)
- moved REF_VOLT_1 39.0 mm to (151.2, 72.5)
- moved R37 35.1 mm to (142.2, 72.8), turned to 90 degrees
- moved C12 30.6 mm to (151.2, 93.5), turned to 180 degrees
- moved RZ_TEMP1 30.5 mm to (178.7, 78.2), turned to 90 degrees
- moved RZ1 30.3 mm to (173.4, 84.7), turned to 0 degrees
- moved TP3 30.1 mm to (146.3, 109.0)
- moved R4 29.8 mm to (151.3, 68.2), turned to 0 degrees
- moved R38 29.1 mm to (167.3, 87.2)
- moved R19 27.5 mm to (151.2, 96.5), turned to 180 degrees
- moved R39 27.0 mm to (167.3, 89.6), turned to 0 degrees
- moved RZ2 25.2 mm to (173.4, 79.7), turned to 180 degrees
- moved REF_PITCH1 23.0 mm to (167.6, 78.3), turned to 90 degrees
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Connections:
- R36 pad 2: REF_VOLT_2 -> REF_PITCH1
- R4 pad 1: Net-(R4-Pad1) -> Net-(REF_VOLT_1-Pad1)
- R4 pad 2: GND -> +5V
- REF_VOLT_1 pad 1: +5V -> Net-(REF_VOLT_1-Pad1)
- Rr2 pad 2: Net-(JP6-Pad2) -> REF_PITCH1
- TP4 pad 1: REF_VOLT_2 -> REF_PITCH1
- U6 pad 1: REF_VOLT_2 -> REF_PITCH1
Routing:
- net +12V: track 0.00 -> 179.1 mm, vias 0 -> 4
- net -12V: track 0.00 -> 136.7 mm, vias 0 -> 2
- net /Inputs/Frequency Control: track 0.00 -> 106.4 mm, vias 0 -> 6
- net +5V: track 0.00 -> 104.1 mm, vias 0 -> 3
- net /Inputs/Scale: track 0.00 -> 79.0 mm, vias 0 -> 1
- net /Inputs/Hard Sync: track 0.00 -> 38.7 mm, vias 0 -> 2
- net REF_VOLT_1: track 0.00 -> 36.4 mm
- net /Outputs/Triangle Output: track 0.00 -> 35.6 mm, vias 0 -> 1
- net Net-(R14-Pad2): track 0.00 -> 34.6 mm
- net /Inputs/Soft Sync: track 0.00 -> 32.7 mm
- net -5V: track 0.00 -> 28.5 mm
- net /Inputs/High Frequency Track: track 0.00 -> 27.9 mm
- net Net-(R28-Pad1): track 0.00 -> 27.4 mm, vias 0 -> 1
- net Net-(R6-Pad2): track 0.00 -> 25.4 mm, vias 0 -> 2
- net /Inputs/Linear FM: track 0.00 -> 23.1 mm, vias 0 -> 1
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Other:
- board text added: "TL074"
- board text removed: "1. RZ_TEMP until TP1-TP2=0V"
- board text removed: "2. Short JP4, C6 with REF_PITCH"
- board text removed: "3. 5V CV, C6 with REFIND_C6"
- board text removed: "4. 0V CV, C0 via Scale ADJ"
- board text removed: "move pots to front"
