File: vco_as3340_v1/vco_as3340.kicad_pcb (KiCad board)
At the start: 2 copper layers, 49 x 100 mm, 100 parts, among them J1 FREQ_CV2, J100 FREQ_CV, J101 SYNC, J102 SAWTOOTH, J103 TRIANGLE, J104 PULSE, J2 Conn_02x05_Odd_Even, U1 LM7805_TO220, U2 L7905, U3 AS3340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

Commit message: Changes to v2 from testing
Parts:
- added C13: 10pF, Capacitor_SMD:C_1206_3216Metric_Pad1.33x1.80mm_HandSolder, B.Cu at (170.2, 135.0)
- added C17: 10pF, Capacitor_SMD:C_1206_3216Metric_Pad1.33x1.80mm_HandSolder, B.Cu at (167.1, 116.6)
- added JP1: Jumper_2_Open, Jumper:SolderJumper-2_P1.3mm_Open_Pad1.0x1.5mm, F.Cu at (155.0, 117.5)
- added R40: 2.5k, Resistor_SMD:R_1206_3216Metric_Pad1.30x1.75mm_HandSolder, B.Cu at (180.3, 99.1)
- added R41: 0, Resistor_SMD:R_1206_3216Metric_Pad1.30x1.75mm_HandSolder, B.Cu at (179.0, 106.9)
- C19: value 10nF -> 10pF
- R21: value 5.1k -> 10k
- R23: value 5.1k -> 0
- R33: value DNU -> 100k
- R34, R4: value 0 -> 100k
- R8: value 100k -> 110k
- Rr1: value 330k -> 220k
- moved C19 31.2 mm to (183.3, 134.2)
- moved R15 3.42 mm to (163.3, 137.5)
Connections:
- C19 pad 1: GND -> Net-(C19-Pad1)
- C19 pad 2: /Inputs/Soft Sync -> Net-(C19-Pad2)
- R25 pad 1: Net-(R25-Pad1) -> Net-(C19-Pad1)
- R27 pad 1: Net-(R27-Pad1) -> Net-(C19-Pad2)
- R27 pad 2: Net-(R25-Pad1) -> Net-(C19-Pad1)
- R29 pad 1: Net-(R27-Pad1) -> Net-(C19-Pad2)
- REFIND_C6 pad 1: +12V -> REF_PITCH1
- RT1 pad 2: VEE -> -5V
- RV_PWM1 pad 1: GND -> Net-(R41-Pad2)
- RV_PWM1 pad 3: +5V -> Net-(R40-Pad1)
- RZ2 pad 2: VEE -> -5V
- SW_SYNC1 pad 1: /Inputs/Soft Sync -> Net-(SW_SYNC1-Pad1)
- U4 pad 6: Net-(R25-Pad1) -> Net-(C19-Pad1)
- U4 pad 7: Net-(R27-Pad1) -> Net-(C19-Pad2)
Routing:
- net -5V: track 28.5 -> 54.2 mm, vias 0 -> 2
- net REF_PITCH1: track 7.27 -> 31.5 mm, vias 0 -> 1
- net +12V: track 179.1 -> 157.7 mm
- net Net-(C19-Pad2): track 0.00 -> 14.1 mm
- net Net-(R27-Pad1): track 13.1 -> 0.00 mm
- net Net-(R41-Pad2): track 0.00 -> 11.3 mm, vias 0 -> 1
- net /Inputs/Soft Sync: track 32.7 -> 21.7 mm
- net Net-(C13-Pad1): track 5.38 -> 14.3 mm
- net Net-(R40-Pad1): track 0.00 -> 7.62 mm, vias 0 -> 1
- net Net-(C19-Pad1): track 0.00 -> 7.33 mm
- net +5V: track 104.1 -> 110.4 mm, vias 3 -> 5
- net VEE: track 5.35 -> 0.00 mm
- net Net-(R25-Pad1): track 5.11 -> 0.00 mm
- net Net-(SW_SYNC1-Pad1): track 0.00 -> 4.10 mm
- net Net-(C13-Pad2): track 16.0 -> 18.7 mm
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Other:
- board text added: "0.1%"
- board text added: "C1 32.70 C2 65.41 C3 130.8 C4 261.6 C5 523.3"
- board text added: "C6 1046.5 C7 2093 C8 4186 C9 8372 C10 16744 C11 33488"
- board text added: "Fine Tune 50% Freq CCW PWM 50% CV 5.000V, REFIND C6 CV 0.000V, ADJ to C1 CV 0.000V, HF to C11"
- board text added: "REFVOLT, 3.75V TP3 REFPITCH, 9.7V TP4 TEMP1, 0V on TP1 TP2 Short J4, C6 w/ REFPITCH"
- board text added: "v2.1 Jan 2023"
- board text removed: "v2.0 Nov 2022"
